Commit message: basicmicro controller

File: urdf/vention.urdf (robot description, URDF)
Before this commit: robot my_robot, 2 links, 1 joints
Links:
- added link vention_base_cam_1_link
Joints:
- added joint vention_base_link_to_vention_base_cam_1: type fixed, parent vention_base_link, child vention_base_cam_1_link, origin xyz=0.3176 0.0 0.386 rpy=0.0 0.0 0.0

Commit message: Debug state

File: urdf/vention.urdf (robot description, URDF)
Before this commit: robot my_robot, 3 links, 2 joints
Links:
- added link zed_mini_base_link
Joints:
- added joint zed_base_link_to_vention_base_link: type fixed, parent zed_mini_base_link, child vention_base_link, origin xyz=-0.3176 0.0 -0.386 rpy=0.0 0.0 0.0
